Commit message: 终于机械臂1指挥了

File: catkin_ws/src/robot/universal_robot/ur_description/urdf/ur5_robotiq85_gripper.urdf copy.xacro (robot description, xacro)
@@ -6,5 +6,5 @@
   <!--  + Height added by the coupler: 8mm -->
   <!--  + Reference frame: at the middle (4mm) -->
-  <!-- <link name="robotiq_coupler">
+  <link name="robotiq_coupler">
     <visual>
       <geometry>
@@ -34,5 +34,5 @@
     <mu2>0.9</mu2>
     <material>Gazebo/FlatBlack</material>
-  </gazebo> -->
+  </gazebo>
   <!-- Equivalent to the OpenRAVE manipulator denso_robotiq_85_gripper -->
   <!-- <link name="denso_robotiq_85_gripper" /> -->
@@ -43,6 +43,6 @@
   <!-- </joint> -->
   <!-- Attach the robotiq 85 gripper -->
-  <xacro:robotiq_85_gripper prefix="" parent="ee_link" >
-    <origin xyz="0 0 0" rpy="0 0 0"/>
+  <xacro:robotiq_85_gripper prefix="" parent="robotiq_coupler" >
+    <origin xyz="0 0 0.004" rpy="0 ${-pi/2} ${pi}"/>
   </xacro:robotiq_85_gripper>
   <!-- Gazebo FT sensor plugin -->
